File: Sens_Board/Sens_Board.kicad_sch (KiCad schematic)
At the start: 2 parts, among them J2 Conn_01x09_Pin, J9 Conn_01x09_Pin

Commit message: Senssoard Firsat LAyout start
Parts:
- J1: renamed from J9; footprint (none) -> Connector_JST:JST_PH_B8B-PH-SM4-TB_1x08-1MP_P2.00mm_Vertical
- J2: footprint (none) -> Connector_JST:JST_PH_B8B-PH-SM4-TB_1x08-1MP_P2.00mm_Vertical
Other:
- moved on the sheet: J2

Commit message: finish SensBoard
Parts:
- added H1, H2: MountingHole, MountingHole:MountingHole_3.2mm_M3, symbol Mechanical:MountingHole
- J1, J2: footprint Connector_JST:JST_PH_B8B-PH-SM4-TB_1x08-1MP_P2.00mm_Vertical -> Connector_JST:JST_PH_B9B-PH-SM4-TB_1x09-1MP_P2.00mm_Vertical
Connections:
- net +5V: now also J2.9 (Pin_9); no longer J2.1 (Pin_1)
- net Data_Clk: now also J2.6 (Pin_6); no longer J2.4 (Pin_4)
- net Data_Latch: now also J2.7 (Pin_7); no longer J2.3 (Pin_3)
- net Data_Output: now also J2.8 (Pin_8); no longer J2.2 (Pin_2)
- net GND: now also J2.1 (Pin_1); no longer J2.9 (Pin_9)
- net Led_Clk: now also J2.2 (Pin_2); no longer J2.8 (Pin_8)
- net Led_Latch: now also J2.3 (Pin_3); no longer J2.7 (Pin_7)
- net Led_OE: now also J2.4 (Pin_4); no longer J2.6 (Pin_6)
Other:
- moved on the sheet: J2
