File: Sens_Board/RJ45.kicad_sch (KiCad schematic)
At the start: 6 parts, among them J3 RJ45_LED_Shielded, J4 RJ45_LED_Shielded, J5 RJ45_LED_Shielded, J6 RJ45_LED_Shielded, J7 RJ45_LED_Shielded, J8 RJ45_LED_Shielded

Commit message: Senssoard Firsat LAyout start
Parts:
- removed J3, J4, J5, J6, J7, J8: RJ45_LED_Shielded, symbol Connector:RJ45_LED_Shielded
- added J3: (no value), LCSC:RJ45-TH_RJ45-TH_HC-RJ45-059D-2X6-2-04, symbol Techbeard:RJ45-12
Connections:
- net GND: now also J3., J3., J3., J3., J3., J3., J3., J3., J3., J3., J3., J3.
- net J3A_Data: now also J3.
- net J3A_Link: now also J3.
- net J3B_Data: now also J3.
- net J3B_Link: now also J3.
- net J3C_Data: now also J3.
- net J3C_Link: now also J3.
- net J3D_Data: now also J3.
- net J3D_Link: now also J3.
- net J3E_Data: now also J3.
- net J3E_Link: now also J3.
- net J3F_Data: now also J3.
- net J3F_Link: now also J3.
- net J3G_Data: now also J3.
- net J3G_Link: now also J3.
- net J3H_Data: now also J3.
- net J3H_Link: now also J3.
- net J3I_Data: now also J3.
- net J3I_Link: now also J3.
- net J3J_Data: now also J3.
- net J3J_Link: now also J3.
- net J3K_Data: now also J3.
- net J3K_Link: now also J3.
- net J3L_Data: now also J3.
- net J3L_Link: now also J3.
- net SchieberegisterInput/D0: now also J3.8
- net SchieberegisterInput/D1: now also J3.7
- net SchieberegisterInput/D2: now also J3.6
- net SchieberegisterInput/D3: now also J3.5
- net SchieberegisterInput/D4: now also J3.4
- net SchieberegisterInput/D5: now also J3.3
- net SchieberegisterInput/D6: now also J3.2
- net SchieberegisterInput/D7: now also J3.1
- net SchieberegisterInput1/D0: now also J3.16
- net SchieberegisterInput1/D1: now also J3.15
- net SchieberegisterInput1/D2: now also J3.14
- net SchieberegisterInput1/D3: now also J3.13
- net SchieberegisterInput1/D4: now also J3.12
- net SchieberegisterInput1/D5: now also J3.11
- net SchieberegisterInput1/D6: now also J3.10
- net SchieberegisterInput1/D7: now also J3.9
- net SchieberegisterInput10/D0: now also J3.128
- net SchieberegisterInput10/D1: now also J3.127
- net SchieberegisterInput10/D2: now also J3.126
- net SchieberegisterInput10/D3: now also J3.125
- net SchieberegisterInput10/D4: now also J3.124
- net SchieberegisterInput10/D5: now also J3.123
- net SchieberegisterInput10/D6: now also J3.122
- net SchieberegisterInput10/D7: now also J3.121
- net SchieberegisterInput11/D0: now also J3.136
- net SchieberegisterInput11/D1: now also J3.135
- net SchieberegisterInput11/D2: now also J3.134
- net SchieberegisterInput11/D3: now also J3.133
- net SchieberegisterInput11/D4: now also J3.132
- net SchieberegisterInput11/D5: now also J3.131
- net SchieberegisterInput11/D6: now also J3.130
- net SchieberegisterInput11/D7: now also J3.129
- net SchieberegisterInput2/D0: now also J3.32
- net SchieberegisterInput2/D1: now also J3.31
- net SchieberegisterInput2/D2: now also J3.30
- net SchieberegisterInput2/D3: now also J3.29
- net SchieberegisterInput2/D4: now also J3.28
- net SchieberegisterInput2/D5: now also J3.27
- net SchieberegisterInput2/D6: now also J3.26
- net SchieberegisterInput2/D7: now also J3.25
- net SchieberegisterInput3/D0: now also J3.40
- net SchieberegisterInput3/D1: now also J3.39
- net SchieberegisterInput3/D2: now also J3.38
- net SchieberegisterInput3/D3: now also J3.37
- net SchieberegisterInput3/D4: now also J3.36
- net SchieberegisterInput3/D5: now also J3.35
- net SchieberegisterInput3/D6: now also J3.34
- net SchieberegisterInput3/D7: now also J3.33
- net SchieberegisterInput4/D0: now also J3.56
- net SchieberegisterInput4/D1: now also J3.55
- net SchieberegisterInput4/D2: now also J3.54
- net SchieberegisterInput4/D3: now also J3.53
- net SchieberegisterInput4/D4: now also J3.52
- net SchieberegisterInput4/D5: now also J3.51
- net SchieberegisterInput4/D6: now also J3.50
- net SchieberegisterInput4/D7: now also J3.49
- net SchieberegisterInput5/D0: now also J3.64
- net SchieberegisterInput5/D1: now also J3.63
- net SchieberegisterInput5/D2: now also J3.62
- net SchieberegisterInput5/D3: now also J3.61
- net SchieberegisterInput5/D4: now also J3.60
- net SchieberegisterInput5/D5: now also J3.59
- net SchieberegisterInput5/D6: now also J3.58
- net SchieberegisterInput5/D7: now also J3.57
- net SchieberegisterInput6/D0: now also J3.80
- net SchieberegisterInput6/D1: now also J3.79
- net SchieberegisterInput6/D2: now also J3.78
- net SchieberegisterInput6/D3: now also J3.77
- net SchieberegisterInput6/D4: now also J3.76
- net SchieberegisterInput6/D5: now also J3.75
- net SchieberegisterInput6/D6: now also J3.74
- net SchieberegisterInput6/D7: now also J3.73
- net SchieberegisterInput7/D0: now also J3.88
- net SchieberegisterInput7/D1: now also J3.87
- net SchieberegisterInput7/D2: now also J3.86
- net SchieberegisterInput7/D3: now also J3.85
- net SchieberegisterInput7/D4: now also J3.84
- net SchieberegisterInput7/D5: now also J3.83
- net SchieberegisterInput7/D6: now also J3.82
- net SchieberegisterInput7/D7: now also J3.81
- net SchieberegisterInput8/D0: now also J3.104
- net SchieberegisterInput8/D1: now also J3.103
- net SchieberegisterInput8/D2: now also J3.102
- net SchieberegisterInput8/D3: now also J3.101
- net SchieberegisterInput8/D4: now also J3.100
- net SchieberegisterInput8/D5: now also J3.99
- net SchieberegisterInput8/D6: now also J3.98
- net SchieberegisterInput8/D7: now also J3.97
- net SchieberegisterInput9/D0: now also J3.112
- net SchieberegisterInput9/D1: now also J3.111
- net SchieberegisterInput9/D2: now also J3.110
- net SchieberegisterInput9/D3: now also J3.109
- net SchieberegisterInput9/D4: now also J3.108
- net SchieberegisterInput9/D5: now also J3.107
- net SchieberegisterInput9/D6: now also J3.106
- net SchieberegisterInput9/D7: now also J3.105

Commit message: finish SensBoard
Connections:
- net GND: now also J3.A11, J3.A9, J3.B11, J3.B9, J3.C11, J3.C9, J3.D11, J3.D9, J3.E11, J3.E9, J3.F12, J3.F9, J3.G11, J3.G9, J3.H11, J3.H9, J3.I11, J3.I9, J3.J11, J3.J9, J3.K11, J3.K9, J3.L11, J3.L9; no longer J3., J3., J3., J3., J3., J3., J3., J3., J3., J3., J3., J3.
- net J3A_Data: now also J3.A10; no longer J3.
- net J3A_Link: now also J3.A12; no longer J3.
- net J3B_Data: now also J3.B10; no longer J3.
- net J3B_Link: now also J3.B12; no longer J3.
- net J3C_Data: now also J3.C10; no longer J3.
- net J3C_Link: now also J3.C12; no longer J3.
- net J3D_Data: now also J3.D10; no longer J3.
- net J3D_Link: now also J3.D12; no longer J3.
- net J3E_Data: now also J3.E10; no longer J3.
- net J3E_Link: now also J3.E12; no longer J3.
- net J3F_Data: now also J3.F10; no longer J3.
- net J3F_Link: now also J3.F13; no longer J3.
- net J3G_Data: now also J3.G10; no longer J3.
- net J3G_Link: now also J3.G12; no longer J3.
- net J3H_Data: now also J3.H10; no longer J3.
- net J3H_Link: now also J3.H12; no longer J3.
- net J3I_Data: now also J3.I10; no longer J3.
- net J3I_Link: now also J3.I12; no longer J3.
- net J3J_Data: now also J3.J10; no longer J3.
- net J3J_Link: now also J3.J12; no longer J3.
- net J3K_Data: now also J3.K10; no longer J3.
- net J3K_Link: now also J3.K12; no longer J3.
- net J3L_Data: now also J3.L10; no longer J3.
- net J3L_Link: now also J3.L12; no longer J3.
- net SchieberegisterInput/D0: now also J3.A8; no longer J3.8
- net SchieberegisterInput/D1: now also J3.A7; no longer J3.7
- net SchieberegisterInput/D2: now also J3.A6; no longer J3.6
- net SchieberegisterInput/D3: now also J3.A5; no longer J3.5
- net SchieberegisterInput/D4: now also J3.A4; no longer J3.4
- net SchieberegisterInput/D5: now also J3.A3; no longer J3.3
- net SchieberegisterInput/D6: now also J3.A2; no longer J3.2
- net SchieberegisterInput/D7: now also J3.A1; no longer J3.1
- net SchieberegisterInput1/D0: now also J3.B8; no longer J3.16
- net SchieberegisterInput1/D1: now also J3.B7; no longer J3.15
- net SchieberegisterInput1/D2: now also J3.B6; no longer J3.14
- net SchieberegisterInput1/D3: now also J3.B5; no longer J3.13
- net SchieberegisterInput1/D4: now also J3.B4; no longer J3.12
- net SchieberegisterInput1/D5: now also J3.B3; no longer J3.11
- net SchieberegisterInput1/D6: now also J3.B2; no longer J3.10
- net SchieberegisterInput1/D7: now also J3.B1; no longer J3.9
- net SchieberegisterInput10/D0: now also J3.K8; no longer J3.128
- net SchieberegisterInput10/D1: now also J3.K7; no longer J3.127
- net SchieberegisterInput10/D2: now also J3.K6; no longer J3.126
- net SchieberegisterInput10/D3: now also J3.K5; no longer J3.125
- net SchieberegisterInput10/D4: now also J3.K4; no longer J3.124
- net SchieberegisterInput10/D5: now also J3.K3; no longer J3.123
- net SchieberegisterInput10/D6: now also J3.K2; no longer J3.122
- net SchieberegisterInput10/D7: now also J3.K1; no longer J3.121
- net SchieberegisterInput11/D0: now also J3.L8; no longer J3.136
- net SchieberegisterInput11/D1: now also J3.L7; no longer J3.135
- net SchieberegisterInput11/D2: now also J3.L6; no longer J3.134
- net SchieberegisterInput11/D3: now also J3.L5; no longer J3.133
- net SchieberegisterInput11/D4: now also J3.L4; no longer J3.132
- net SchieberegisterInput11/D5: now also J3.L3; no longer J3.131
- net SchieberegisterInput11/D6: now also J3.L2; no longer J3.130
- net SchieberegisterInput11/D7: now also J3.L1; no longer J3.129
- net SchieberegisterInput2/D0: now also J3.C8; no longer J3.32
- net SchieberegisterInput2/D1: now also J3.C7; no longer J3.31
- net SchieberegisterInput2/D2: now also J3.C6; no longer J3.30
- net SchieberegisterInput2/D3: now also J3.C5; no longer J3.29
- net SchieberegisterInput2/D4: now also J3.C4; no longer J3.28
- net SchieberegisterInput2/D5: now also J3.C3; no longer J3.27
- net SchieberegisterInput2/D6: now also J3.C2; no longer J3.26
- net SchieberegisterInput2/D7: now also J3.C1; no longer J3.25
- net SchieberegisterInput3/D0: now also J3.D8; no longer J3.40
- net SchieberegisterInput3/D1: now also J3.D7; no longer J3.39
- net SchieberegisterInput3/D2: now also J3.D6; no longer J3.38
- net SchieberegisterInput3/D3: now also J3.D5; no longer J3.37
- net SchieberegisterInput3/D4: now also J3.D4; no longer J3.36
- net SchieberegisterInput3/D5: now also J3.D3; no longer J3.35
- net SchieberegisterInput3/D6: now also J3.D2; no longer J3.34
- net SchieberegisterInput3/D7: now also J3.D1; no longer J3.33
- net SchieberegisterInput4/D0: now also J3.E8; no longer J3.56
- net SchieberegisterInput4/D1: now also J3.E7; no longer J3.55
- net SchieberegisterInput4/D2: now also J3.E6; no longer J3.54
- net SchieberegisterInput4/D3: now also J3.E5; no longer J3.53
- net SchieberegisterInput4/D4: now also J3.E4; no longer J3.52
- net SchieberegisterInput4/D5: now also J3.E3; no longer J3.51
- net SchieberegisterInput4/D6: now also J3.E2; no longer J3.50
- net SchieberegisterInput4/D7: now also J3.E1; no longer J3.49
- net SchieberegisterInput5/D0: now also J3.F8; no longer J3.64
- net SchieberegisterInput5/D1: now also J3.F7; no longer J3.63
- net SchieberegisterInput5/D2: now also J3.F6; no longer J3.62
- net SchieberegisterInput5/D3: now also J3.F5; no longer J3.61
- net SchieberegisterInput5/D4: now also J3.F4; no longer J3.60
- net SchieberegisterInput5/D5: now also J3.F3; no longer J3.59
- net SchieberegisterInput5/D6: now also J3.F2; no longer J3.58
- net SchieberegisterInput5/D7: now also J3.F1; no longer J3.57
- net SchieberegisterInput6/D0: now also J3.G8; no longer J3.80
- net SchieberegisterInput6/D1: now also J3.G7; no longer J3.79
- net SchieberegisterInput6/D2: now also J3.G6; no longer J3.78
- net SchieberegisterInput6/D3: now also J3.G5; no longer J3.77
- net SchieberegisterInput6/D4: now also J3.G4; no longer J3.76
- net SchieberegisterInput6/D5: now also J3.G3; no longer J3.75
- net SchieberegisterInput6/D6: now also J3.G2; no longer J3.74
- net SchieberegisterInput6/D7: now also J3.G1; no longer J3.73
- net SchieberegisterInput7/D0: now also J3.H8; no longer J3.88
- net SchieberegisterInput7/D1: now also J3.H7; no longer J3.87
- net SchieberegisterInput7/D2: now also J3.H6; no longer J3.86
- net SchieberegisterInput7/D3: now also J3.H5; no longer J3.85
- net SchieberegisterInput7/D4: now also J3.H4; no longer J3.84
- net SchieberegisterInput7/D5: now also J3.H3; no longer J3.83
- net SchieberegisterInput7/D6: now also J3.H2; no longer J3.82
- net SchieberegisterInput7/D7: now also J3.H1; no longer J3.81
- net SchieberegisterInput8/D0: now also J3.I8; no longer J3.104
- net SchieberegisterInput8/D1: now also J3.I7; no longer J3.103
- net SchieberegisterInput8/D2: now also J3.I6; no longer J3.102
- net SchieberegisterInput8/D3: now also J3.I5; no longer J3.101
- net SchieberegisterInput8/D4: now also J3.I4; no longer J3.100
- net SchieberegisterInput8/D5: now also J3.I3; no longer J3.99
- net SchieberegisterInput8/D6: now also J3.I2; no longer J3.98
- net SchieberegisterInput8/D7: now also J3.I1; no longer J3.97
- net SchieberegisterInput9/D0: now also J3.J8; no longer J3.112
- net SchieberegisterInput9/D1: now also J3.J7; no longer J3.111
- net SchieberegisterInput9/D2: now also J3.J6; no longer J3.110
- net SchieberegisterInput9/D3: now also J3.J5; no longer J3.109
- net SchieberegisterInput9/D4: now also J3.J4; no longer J3.108
- net SchieberegisterInput9/D5: now also J3.J3; no longer J3.107
- net SchieberegisterInput9/D6: now also J3.J2; no longer J3.106
- net SchieberegisterInput9/D7: now also J3.J1; no longer J3.105

Commit message: fixes and optmierung
Connections:
- net SchieberegisterInput/D0: now also J3.A5; no longer J3.A8
- net SchieberegisterInput/D1: now also J3.A6; no longer J3.A7
- net SchieberegisterInput/D2: now also J3.A7; no longer J3.A6
- net SchieberegisterInput/D3: now also J3.A8; no longer J3.A5
- net SchieberegisterInput/D4: now also J3.A1; no longer J3.A4
- net SchieberegisterInput/D5: now also J3.A2; no longer J3.A3
- net SchieberegisterInput/D6: now also J3.A3; no longer J3.A2
- net SchieberegisterInput/D7: now also J3.A4; no longer J3.A1
- net SchieberegisterInput1/D0: now also J3.B5; no longer J3.B8
- net SchieberegisterInput1/D1: now also J3.B6; no longer J3.B7
- net SchieberegisterInput1/D2: now also J3.B7; no longer J3.B6
- net SchieberegisterInput1/D3: now also J3.B8; no longer J3.B5
- net SchieberegisterInput1/D4: now also J3.B1; no longer J3.B4
- net SchieberegisterInput1/D5: now also J3.B2; no longer J3.B3
- net SchieberegisterInput1/D6: now also J3.B3; no longer J3.B2
- net SchieberegisterInput1/D7: now also J3.B4; no longer J3.B1
- net SchieberegisterInput10/D0: now also J3.K5; no longer J3.K8
- net SchieberegisterInput10/D1: now also J3.K6; no longer J3.K7
- net SchieberegisterInput10/D2: now also J3.K7; no longer J3.K6
- net SchieberegisterInput10/D3: now also J3.K8; no longer J3.K5
- net SchieberegisterInput10/D4: now also J3.K1; no longer J3.K4
- net SchieberegisterInput10/D5: now also J3.K2; no longer J3.K3
- net SchieberegisterInput10/D6: now also J3.K3; no longer J3.K2
- net SchieberegisterInput10/D7: now also J3.K4; no longer J3.K1
- net SchieberegisterInput11/D0: now also J3.L5; no longer J3.L8
- net SchieberegisterInput11/D1: now also J3.L6; no longer J3.L7
- net SchieberegisterInput11/D2: now also J3.L7; no longer J3.L6
- net SchieberegisterInput11/D3: now also J3.L8; no longer J3.L5
- net SchieberegisterInput11/D4: now also J3.L1; no longer J3.L4
- net SchieberegisterInput11/D5: now also J3.L2; no longer J3.L3
- net SchieberegisterInput11/D6: now also J3.L3; no longer J3.L2
- net SchieberegisterInput11/D7: now also J3.L4; no longer J3.L1
- net SchieberegisterInput2/D0: now also J3.C5; no longer J3.C8
- net SchieberegisterInput2/D1: now also J3.C6; no longer J3.C7
- net SchieberegisterInput2/D2: now also J3.C7; no longer J3.C6
- net SchieberegisterInput2/D3: now also J3.C8; no longer J3.C5
- net SchieberegisterInput2/D4: now also J3.C1; no longer J3.C4
- net SchieberegisterInput2/D5: now also J3.C2; no longer J3.C3
- net SchieberegisterInput2/D6: now also J3.C3; no longer J3.C2
- net SchieberegisterInput2/D7: now also J3.C4; no longer J3.C1
- net SchieberegisterInput3/D0: now also J3.D5; no longer J3.D8
- net SchieberegisterInput3/D1: now also J3.D6; no longer J3.D7
- net SchieberegisterInput3/D2: now also J3.D7; no longer J3.D6
- net SchieberegisterInput3/D3: now also J3.D8; no longer J3.D5
- net SchieberegisterInput3/D4: now also J3.D1; no longer J3.D4
- net SchieberegisterInput3/D5: now also J3.D2; no longer J3.D3
- net SchieberegisterInput3/D6: now also J3.D3; no longer J3.D2
- net SchieberegisterInput3/D7: now also J3.D4; no longer J3.D1
- net SchieberegisterInput4/D0: now also J3.E5; no longer J3.E8
- net SchieberegisterInput4/D1: now also J3.E6; no longer J3.E7
- net SchieberegisterInput4/D2: now also J3.E7; no longer J3.E6
- net SchieberegisterInput4/D3: now also J3.E8; no longer J3.E5
- net SchieberegisterInput4/D4: now also J3.E1; no longer J3.E4
- net SchieberegisterInput4/D5: now also J3.E2; no longer J3.E3
- net SchieberegisterInput4/D6: now also J3.E3; no longer J3.E2
- net SchieberegisterInput4/D7: now also J3.E4; no longer J3.E1
- net SchieberegisterInput5/D0: now also J3.F5; no longer J3.F8
- net SchieberegisterInput5/D1: now also J3.F6; no longer J3.F7
- net SchieberegisterInput5/D2: now also J3.F7; no longer J3.F6
- net SchieberegisterInput5/D3: now also J3.F8; no longer J3.F5
- net SchieberegisterInput5/D4: now also J3.F1; no longer J3.F4
- net SchieberegisterInput5/D5: now also J3.F2; no longer J3.F3
- net SchieberegisterInput5/D6: now also J3.F3; no longer J3.F2
- net SchieberegisterInput5/D7: now also J3.F4; no longer J3.F1
- net SchieberegisterInput6/D0: now also J3.G5; no longer J3.G8
- net SchieberegisterInput6/D1: now also J3.G6; no longer J3.G7
- net SchieberegisterInput6/D2: now also J3.G7; no longer J3.G6
- net SchieberegisterInput6/D3: now also J3.G8; no longer J3.G5
- net SchieberegisterInput6/D4: now also J3.G1; no longer J3.G4
- net SchieberegisterInput6/D5: now also J3.G2; no longer J3.G3
- net SchieberegisterInput6/D6: now also J3.G3; no longer J3.G2
- net SchieberegisterInput6/D7: now also J3.G4; no longer J3.G1
- net SchieberegisterInput7/D0: now also J3.H5; no longer J3.H8
- net SchieberegisterInput7/D1: now also J3.H6; no longer J3.H7
- net SchieberegisterInput7/D2: now also J3.H7; no longer J3.H6
- net SchieberegisterInput7/D3: now also J3.H8; no longer J3.H5
- net SchieberegisterInput7/D4: now also J3.H1; no longer J3.H4
- net SchieberegisterInput7/D5: now also J3.H2; no longer J3.H3
- net SchieberegisterInput7/D6: now also J3.H3; no longer J3.H2
- net SchieberegisterInput7/D7: now also J3.H4; no longer J3.H1
- net SchieberegisterInput8/D0: now also J3.I5; no longer J3.I8
- net SchieberegisterInput8/D1: now also J3.I6; no longer J3.I7
- net SchieberegisterInput8/D2: now also J3.I7; no longer J3.I6
- net SchieberegisterInput8/D3: now also J3.I8; no longer J3.I5
- net SchieberegisterInput8/D4: now also J3.I1; no longer J3.I4
- net SchieberegisterInput8/D5: now also J3.I2; no longer J3.I3
- net SchieberegisterInput8/D6: now also J3.I3; no longer J3.I2
- net SchieberegisterInput8/D7: now also J3.I4; no longer J3.I1
- net SchieberegisterInput9/D0: now also J3.J5; no longer J3.J8
- net SchieberegisterInput9/D1: now also J3.J6; no longer J3.J7
- net SchieberegisterInput9/D2: now also J3.J7; no longer J3.J6
- net SchieberegisterInput9/D3: now also J3.J8; no longer J3.J5
- net SchieberegisterInput9/D4: now also J3.J1; no longer J3.J4
- net SchieberegisterInput9/D5: now also J3.J2; no longer J3.J3
- net SchieberegisterInput9/D6: now also J3.J3; no longer J3.J2
- net SchieberegisterInput9/D7: now also J3.J4; no longer J3.J1

Commit message: Production File generate
Connections:
- net GND: now also J3.F11; no longer J3.F12
- net J3F_Link: now also J3.F12; no longer J3.F13
Changed lines of the file:
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@@
 	)
 	(symbol
+		(lib_name "RJ45-12_1")
 		(lib_id "Techbeard:RJ45-12")
 		(at 100.33 86.36 0)
@@
 		(pin "B7"
 		)
-		(pin "F13"
+		(pin "F11"
 		)
 		(pin "E12"
