File: Sens_Board/Sens_Board.kicad_pcb (KiCad board)
At the start: 4 copper layers, 200 x 100 mm, 247 parts, among them U1 74HC595, U10 74HC165, U11 74HC165, U12 74HC165, U13 74HC165, U14 74HC165, U15 74HC165, U2 74HC595, U22 RJ45_Amphenol_54602-x08_Horiz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, U3 74HC595, U4 74HC165, U5 74HC165, U6 74HC165, U7 74HC165, U8 74HC165, U9 74HC165

Commit message: Senssoard Firsat LAyout start
Parts:
- removed R121: R, Resistor_SMD:R_0603_1608Metric
- removed U22: RJ45_Amphenol_54602-x08_Horizontal, Connector_RJ:RJ45_Amphenol_54602-x08_Horizontal
- added J1: Conn_01x09_Pin, Connector_JST:JST_PH_B8B-PH-SM4-TB_1x08-1MP_P2.00mm_Vertical, F.Cu at (88.8, 46.2)
- added J2: Conn_01x09_Pin, Connector_JST:JST_PH_B8B-PH-SM4-TB_1x08-1MP_P2.00mm_Vertical, F.Cu at (90.8, 133.2)
- added J3: ~, LCSC:RJ45-TH_RJ45-TH_HC-RJ45-059D-2X6-2-04, F.Cu at (215.5, 87.4)
- added R9: R, Resistor_SMD:R_0402_1005Metric, F.Cu at (66.2, 69.8)
- C1, C10, C100, C101, C102, C103, C104, C105, C106, C107, C108, C109, C11, C110, C111, C12, C13, C14, C15, C16, C17, C18, C19, C2, C20, C21, C22, C23, C24, C25, C26, C27, C28, C29, C3, C30, C31, C32, C33, C34, C35, C36, C37, C38, C39, C4, C40, C41, C42, C43, C44, C45, C46, C47, C48, C49, C5, C50, C51, C52, C53, C54, C55, C56, C57, C58, C59, C6, C60, C61, C62, C63, C64, C65, C66, C67, C68, C69, C7, C70, C71, C72, C73, C74, C75, C76, C77, C78, C79, C8, C80, C81, C82, C83, C84, C85, C86, C87, C88, C89, C9, C90, C91, C92, C93, C94, C95, C96, C97, C98, C99: footprint Capacitor_SMD:C_0603_1608Metric -> Capacitor_SMD:C_0402_1005Metric
- R1, R10, R100, R101, R102, R103, R104, R105, R106, R107, R108, R109, R11, R110, R111, R112, R113, R12, R13, R14, R15, R16, R17, R2, R25, R26, R27, R28, R29, R3, R30, R31, R32, R33, R34, R35, R36, R37, R38, R39, R4, R40, R41, R42, R43, R44, R45, R46, R47, R48, R49, R5, R50, R51, R52, R53, R54, R55, R56, R57, R58, R59, R6, R60, R61, R62, R63, R64, R65, R66, R67, R68, R69, R7, R70, R71, R72, R73, R74, R75, R76, R77, R78, R79, R8, R80, R81, R82, R83, R84, R85, R86, R87, R88, R89, R90, R91, R92, R93, R94, R95, R96, R97, R98, R99: footprint Resistor_SMD:R_0603_1608Metric -> Resistor_SMD:R_0402_1005Metric
- R114, R115, R116, R117, R118, R119, R120: value R -> 10k; footprint Resistor_SMD:R_0603_1608Metric -> Resistor_SMD:R_0402_1005Metric
- R18, R19, R20, R21, R22, R23, R24: value 10k -> R; footprint Resistor_SMD:R_0603_1608Metric -> Resistor_SMD:R_0402_1005Metric
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Connections:
- C10 pad 1: +5V -> /RJ45/SchieberegisterInput/D2
- C100 pad 1: unconnected-(C100-Pad1) -> /RJ45/SchieberegisterInput10/D2
- C101 pad 1: unconnected-(C101-Pad1) -> /RJ45/SchieberegisterInput10/D1
- C102 pad 1: unconnected-(C102-Pad1) -> /RJ45/SchieberegisterInput10/D0
- C103 pad 1: unconnected-(C103-Pad1) -> +5V
- C104 pad 1: unconnected-(C104-Pad1) -> /RJ45/SchieberegisterInput11/D7
- C105 pad 1: unconnected-(C105-Pad1) -> /RJ45/SchieberegisterInput11/D6
- C106 pad 1: unconnected-(C106-Pad1) -> /RJ45/SchieberegisterInput11/D5
- C107 pad 1: unconnected-(C107-Pad1) -> /RJ45/SchieberegisterInput11/D4
- C108 pad 1: unconnected-(C108-Pad1) -> /RJ45/SchieberegisterInput11/D3
- C109 pad 1: unconnected-(C109-Pad1) -> /RJ45/SchieberegisterInput11/D2
- C11 pad 1: +5V -> /RJ45/SchieberegisterInput/D1
- C110 pad 1: unconnected-(C110-Pad1) -> /RJ45/SchieberegisterInput11/D1
- C111 pad 1: unconnected-(C111-Pad1) -> /RJ45/SchieberegisterInput11/D0
- C12 pad 1: +5V -> /RJ45/SchieberegisterInput/D0
- C14 pad 1: +5V -> /RJ45/SchieberegisterInput2/D7
- C15 pad 1: +5V -> /RJ45/SchieberegisterInput2/D6
- C16 pad 1: unconnected-(C16-Pad1) -> /RJ45/SchieberegisterInput2/D5
- C17 pad 1: unconnected-(C17-Pad1) -> /RJ45/SchieberegisterInput2/D4
- C18 pad 1: unconnected-(C18-Pad1) -> /RJ45/SchieberegisterInput2/D3
- C19 pad 1: unconnected-(C19-Pad1) -> /RJ45/SchieberegisterInput2/D2
- C20 pad 1: unconnected-(C20-Pad1) -> /RJ45/SchieberegisterInput2/D1
- C21 pad 1: unconnected-(C21-Pad1) -> /RJ45/SchieberegisterInput2/D0
- C22 pad 1: unconnected-(C22-Pad1) -> +5V
- C23 pad 1: unconnected-(C23-Pad1) -> /RJ45/SchieberegisterInput1/D7
- C24 pad 1: unconnected-(C24-Pad1) -> /RJ45/SchieberegisterInput1/D6
- C25 pad 1: unconnected-(C25-Pad1) -> /RJ45/SchieberegisterInput1/D5
- C26 pad 1: unconnected-(C26-Pad1) -> /RJ45/SchieberegisterInput1/D4
- C27 pad 1: unconnected-(C27-Pad1) -> /RJ45/SchieberegisterInput1/D3
- C28 pad 1: unconnected-(C28-Pad1) -> /RJ45/SchieberegisterInput1/D2
- C29 pad 1: unconnected-(C29-Pad1) -> /RJ45/SchieberegisterInput1/D1
- C30 pad 1: unconnected-(C30-Pad1) -> /RJ45/SchieberegisterInput1/D0
- C31 pad 1: unconnected-(C31-Pad1) -> +5V
- C32 pad 1: unconnected-(C32-Pad1) -> /RJ45/SchieberegisterInput3/D7
- C33 pad 1: unconnected-(C33-Pad1) -> /RJ45/SchieberegisterInput3/D6
- C34 pad 1: unconnected-(C34-Pad1) -> /RJ45/SchieberegisterInput3/D5
- C35 pad 1: unconnected-(C35-Pad1) -> /RJ45/SchieberegisterInput3/D4
- C36 pad 1: unconnected-(C36-Pad1) -> /RJ45/SchieberegisterInput3/D3
- C37 pad 1: unconnected-(C37-Pad1) -> /RJ45/SchieberegisterInput3/D2
- C38 pad 1: unconnected-(C38-Pad1) -> /RJ45/SchieberegisterInput3/D1
- C39 pad 1: unconnected-(C39-Pad1) -> /RJ45/SchieberegisterInput3/D0
- C40 pad 1: unconnected-(C40-Pad1) -> +5V
- C41 pad 1: unconnected-(C41-Pad1) -> /RJ45/SchieberegisterInput4/D7
- C42 pad 1: unconnected-(C42-Pad1) -> /RJ45/SchieberegisterInput4/D6
- C43 pad 1: unconnected-(C43-Pad1) -> /RJ45/SchieberegisterInput4/D5
- C44 pad 1: unconnected-(C44-Pad1) -> /RJ45/SchieberegisterInput4/D4
- C45 pad 1: unconnected-(C45-Pad1) -> /RJ45/SchieberegisterInput4/D3
- C46 pad 1: unconnected-(C46-Pad1) -> /RJ45/SchieberegisterInput4/D2
- C47 pad 1: unconnected-(C47-Pad1) -> /RJ45/SchieberegisterInput4/D1
- C48 pad 1: unconnected-(C48-Pad1) -> /RJ45/SchieberegisterInput4/D0
- C49 pad 1: unconnected-(C49-Pad1) -> +5V
- C5 pad 1: +5V -> /RJ45/SchieberegisterInput/D7
- C50 pad 1: unconnected-(C50-Pad1) -> /RJ45/SchieberegisterInput5/D7
- C51 pad 1: unconnected-(C51-Pad1) -> /RJ45/SchieberegisterInput5/D6
- C52 pad 1: unconnected-(C52-Pad1) -> /RJ45/SchieberegisterInput5/D5
- C53 pad 1: unconnected-(C53-Pad1) -> /RJ45/SchieberegisterInput5/D4
- C54 pad 1: unconnected-(C54-Pad1) -> /RJ45/SchieberegisterInput5/D3
- C55 pad 1: unconnected-(C55-Pad1) -> /RJ45/SchieberegisterInput5/D2
- C56 pad 1: unconnected-(C56-Pad1) -> /RJ45/SchieberegisterInput5/D1
- C57 pad 1: unconnected-(C57-Pad1) -> /RJ45/SchieberegisterInput5/D0
- C58 pad 1: unconnected-(C58-Pad1) -> +5V
- C59 pad 1: unconnected-(C59-Pad1) -> /RJ45/SchieberegisterInput6/D7
- C6 pad 1: +5V -> /RJ45/SchieberegisterInput/D6
- C60 pad 1: unconnected-(C60-Pad1) -> /RJ45/SchieberegisterInput6/D6
- C61 pad 1: unconnected-(C61-Pad1) -> /RJ45/SchieberegisterInput6/D5
- C62 pad 1: unconnected-(C62-Pad1) -> /RJ45/SchieberegisterInput6/D4
- C63 pad 1: unconnected-(C63-Pad1) -> /RJ45/SchieberegisterInput6/D3
- C64 pad 1: unconnected-(C64-Pad1) -> /RJ45/SchieberegisterInput6/D2
- C65 pad 1: unconnected-(C65-Pad1) -> /RJ45/SchieberegisterInput6/D1
- C66 pad 1: unconnected-(C66-Pad1) -> /RJ45/SchieberegisterInput6/D0
- C67 pad 1: unconnected-(C67-Pad1) -> +5V
- C68 pad 1: unconnected-(C68-Pad1) -> /RJ45/SchieberegisterInput7/D7
- C69 pad 1: unconnected-(C69-Pad1) -> /RJ45/SchieberegisterInput7/D6
- C7 pad 1: +5V -> /RJ45/SchieberegisterInput/D5
- C70 pad 1: unconnected-(C70-Pad1) -> /RJ45/SchieberegisterInput7/D5
- C71 pad 1: unconnected-(C71-Pad1) -> /RJ45/SchieberegisterInput7/D4
- C72 pad 1: unconnected-(C72-Pad1) -> /RJ45/SchieberegisterInput7/D3
- C73 pad 1: unconnected-(C73-Pad1) -> /RJ45/SchieberegisterInput7/D2
- C74 pad 1: unconnected-(C74-Pad1) -> /RJ45/SchieberegisterInput7/D1
- C75 pad 1: unconnected-(C75-Pad1) -> /RJ45/SchieberegisterInput7/D0
- C76 pad 1: unconnected-(C76-Pad1) -> +5V
- C77 pad 1: unconnected-(C77-Pad1) -> /RJ45/SchieberegisterInput8/D7
- C78 pad 1: unconnected-(C78-Pad1) -> /RJ45/SchieberegisterInput8/D6
- C79 pad 1: unconnected-(C79-Pad1) -> /RJ45/SchieberegisterInput8/D5
- C8 pad 1: +5V -> /RJ45/SchieberegisterInput/D4
- C80 pad 1: unconnected-(C80-Pad1) -> /RJ45/SchieberegisterInput8/D4
- C81 pad 1: unconnected-(C81-Pad1) -> /RJ45/SchieberegisterInput8/D3
- C82 pad 1: unconnected-(C82-Pad1) -> /RJ45/SchieberegisterInput8/D2
- C83 pad 1: unconnected-(C83-Pad1) -> /RJ45/SchieberegisterInput8/D1
- C84 pad 1: unconnected-(C84-Pad1) -> /RJ45/SchieberegisterInput8/D0
- C85 pad 1: unconnected-(C85-Pad1) -> +5V
- C86 pad 1: unconnected-(C86-Pad1) -> /RJ45/SchieberegisterInput9/D7
- C87 pad 1: unconnected-(C87-Pad1) -> /RJ45/SchieberegisterInput9/D6
- C88 pad 1: unconnected-(C88-Pad1) -> /RJ45/SchieberegisterInput9/D5
- C89 pad 1: unconnected-(C89-Pad1) -> /RJ45/SchieberegisterInput9/D4
- C9 pad 1: +5V -> /RJ45/SchieberegisterInput/D3
- C90 pad 1: unconnected-(C90-Pad1) -> /RJ45/SchieberegisterInput9/D3
- C91 pad 1: unconnected-(C91-Pad1) -> /RJ45/SchieberegisterInput9/D2
- C92 pad 1: unconnected-(C92-Pad1) -> /RJ45/SchieberegisterInput9/D1
- C93 pad 1: unconnected-(C93-Pad1) -> /RJ45/SchieberegisterInput9/D0
- C94 pad 1: unconnected-(C94-Pad1) -> +5V
- C95 pad 1: unconnected-(C95-Pad1) -> /RJ45/SchieberegisterInput10/D7
- C96 pad 1: unconnected-(C96-Pad1) -> /RJ45/SchieberegisterInput10/D6
- C97 pad 1: unconnected-(C97-Pad1) -> /RJ45/SchieberegisterInput10/D5
- C98 pad 1: unconnected-(C98-Pad1) -> /RJ45/SchieberegisterInput10/D4
- C99 pad 1: unconnected-(C99-Pad1) -> /RJ45/SchieberegisterInput10/D3
- R10 pad 1: Net-(U2-QC) -> Net-(U2-QB)
- R10 pad 2: /OutputShift2/Out2 -> /OutputShift/Out1
- R100 pad 2: /RJ45/SchieberegisterInput9/D5 -> /RJ45/SchieberegisterInput9/D4
- R101 pad 2: /RJ45/SchieberegisterInput9/D4 -> /RJ45/SchieberegisterInput9/D3
- R102 pad 2: /RJ45/SchieberegisterInput9/D3 -> /RJ45/SchieberegisterInput9/D2
- R103 pad 2: /RJ45/SchieberegisterInput9/D2 -> /RJ45/SchieberegisterInput9/D1
- R104 pad 2: /RJ45/SchieberegisterInput9/D1 -> /RJ45/SchieberegisterInput9/D0
- R105 pad 2: /RJ45/SchieberegisterInput9/D0 -> /RJ45/SchieberegisterInput10/D7
- R106 pad 2: /RJ45/SchieberegisterInput11/D7 -> /RJ45/SchieberegisterInput10/D6
- R107 pad 2: /RJ45/SchieberegisterInput11/D6 -> /RJ45/SchieberegisterInput10/D5
- R108 pad 2: /RJ45/SchieberegisterInput11/D5 -> /RJ45/SchieberegisterInput10/D4
- R109 pad 2: /RJ45/SchieberegisterInput11/D4 -> /RJ45/SchieberegisterInput10/D3
- R11 pad 1: Net-(U1-QD) -> Net-(U2-QC)
- R11 pad 2: /OutputShift1/Out3 -> /OutputShift/Out2
- R110 pad 2: /RJ45/SchieberegisterInput11/D3 -> /RJ45/SchieberegisterInput10/D2
- R111 pad 2: /RJ45/SchieberegisterInput11/D2 -> /RJ45/SchieberegisterInput10/D1
- R112 pad 2: /RJ45/SchieberegisterInput11/D1 -> /RJ45/SchieberegisterInput10/D0
- R113 pad 2: /RJ45/SchieberegisterInput11/D0 -> /RJ45/SchieberegisterInput11/D7
- R114 pad 1: Net-(U3-QF) -> +5V
- R114 pad 2: /OutputShift/Out5 -> /RJ45/SchieberegisterInput11/D6
- R115 pad 1: Net-(U2-QF) -> +5V
- R115 pad 2: /OutputShift2/Out5 -> /RJ45/SchieberegisterInput11/D5
- R116 pad 1: Net-(U1-QG) -> +5V
- R116 pad 2: /OutputShift1/Out6 -> /RJ45/SchieberegisterInput11/D4
- R117 pad 1: Net-(U3-QG) -> +5V
- R117 pad 2: /OutputShift/Out6 -> /RJ45/SchieberegisterInput11/D3
- R118 pad 1: Net-(U2-QG) -> +5V
- R118 pad 2: /OutputShift2/Out6 -> /RJ45/SchieberegisterInput11/D2
- R119 pad 1: Net-(U1-QH) -> +5V
- R119 pad 2: /OutputShift1/Out7 -> /RJ45/SchieberegisterInput11/D1
- R12 pad 1: Net-(U3-QD) -> Net-(U2-QD)
- R120 pad 1: Net-(U3-QH) -> +5V
- R120 pad 2: /OutputShift/Out7 -> /RJ45/SchieberegisterInput11/D0
- R13 pad 1: Net-(U2-QD) -> Net-(U2-QE)
- R13 pad 2: /OutputShift2/Out3 -> /OutputShift/Out4
- R14 pad 1: Net-(U1-QE) -> Net-(U2-QF)
- R14 pad 2: /OutputShift1/Out4 -> /OutputShift/Out5
- R15 pad 1: Net-(U3-QE) -> Net-(U2-QG)
- R15 pad 2: /OutputShift/Out4 -> /OutputShift/Out6
- R16 pad 1: Net-(U2-QE) -> Net-(U2-QH)
- R16 pad 2: /OutputShift2/Out4 -> /OutputShift/Out7
- R17 pad 1: Net-(U1-QF) -> Net-(U3-QA)
- R17 pad 2: /OutputShift1/Out5 -> /OutputShift2/Out0
- R18 pad 1: +5V -> Net-(U3-QB)
- R18 pad 2: /RJ45/SchieberegisterInput/D7 -> /OutputShift2/Out1
- R19 pad 1: +5V -> Net-(U3-QC)
- R19 pad 2: /RJ45/SchieberegisterInput/D6 -> /OutputShift2/Out2
- R2 pad 1: Net-(U3-QA) -> Net-(U1-QB)
- R2 pad 2: /OutputShift/Out0 -> /OutputShift1/Out1
- R20 pad 1: +5V -> Net-(U3-QD)
- R20 pad 2: /RJ45/SchieberegisterInput/D5 -> /OutputShift2/Out3
- R21 pad 1: +5V -> Net-(U3-QE)
- R21 pad 2: /RJ45/SchieberegisterInput/D4 -> /OutputShift2/Out4
- R22 pad 1: +5V -> Net-(U3-QF)
- R22 pad 2: /RJ45/SchieberegisterInput/D3 -> /OutputShift2/Out5
- R23 pad 1: +5V -> Net-(U3-QG)
- R23 pad 2: /RJ45/SchieberegisterInput/D2 -> /OutputShift2/Out6
- R24 pad 1: +5V -> Net-(U3-QH)
- R24 pad 2: /RJ45/SchieberegisterInput/D1 -> /OutputShift2/Out7
- R25 pad 2: /RJ45/SchieberegisterInput/D0 -> /RJ45/SchieberegisterInput/D7
- R26 pad 2: /RJ45/SchieberegisterInput2/D7 -> /RJ45/SchieberegisterInput/D6
- R27 pad 2: /RJ45/SchieberegisterInput2/D6 -> /RJ45/SchieberegisterInput/D5
- R28 pad 2: /RJ45/SchieberegisterInput2/D5 -> /RJ45/SchieberegisterInput/D4
- R29 pad 2: /RJ45/SchieberegisterInput2/D4 -> /RJ45/SchieberegisterInput/D3
- R3 pad 1: Net-(U2-QA) -> Net-(U1-QC)
- R3 pad 2: /OutputShift2/Out0 -> /OutputShift1/Out2
- R30 pad 2: /RJ45/SchieberegisterInput2/D3 -> /RJ45/SchieberegisterInput/D2
- R31 pad 2: /RJ45/SchieberegisterInput2/D2 -> /RJ45/SchieberegisterInput/D1
- R32 pad 2: /RJ45/SchieberegisterInput2/D1 -> /RJ45/SchieberegisterInput/D0
- R33 pad 2: /RJ45/SchieberegisterInput2/D0 -> /RJ45/SchieberegisterInput2/D7
- R34 pad 2: /RJ45/SchieberegisterInput1/D7 -> /RJ45/SchieberegisterInput2/D6
- R35 pad 2: /RJ45/SchieberegisterInput1/D6 -> /RJ45/SchieberegisterInput2/D5
- R36 pad 2: /RJ45/SchieberegisterInput1/D5 -> /RJ45/SchieberegisterInput2/D4
- R37 pad 2: /RJ45/SchieberegisterInput1/D4 -> /RJ45/SchieberegisterInput2/D3
- R38 pad 2: /RJ45/SchieberegisterInput1/D3 -> /RJ45/SchieberegisterInput2/D2
- R39 pad 2: /RJ45/SchieberegisterInput1/D2 -> /RJ45/SchieberegisterInput2/D1
- R4 pad 1: Net-(U1-QB) -> Net-(U1-QD)
- R4 pad 2: /OutputShift1/Out1 -> /OutputShift1/Out3
- R40 pad 2: /RJ45/SchieberegisterInput1/D1 -> /RJ45/SchieberegisterInput2/D0
- R41 pad 2: /RJ45/SchieberegisterInput1/D0 -> /RJ45/SchieberegisterInput1/D7
- R42 pad 2: /RJ45/SchieberegisterInput3/D7 -> /RJ45/SchieberegisterInput1/D6
- R43 pad 2: /RJ45/SchieberegisterInput3/D6 -> /RJ45/SchieberegisterInput1/D5
- R44 pad 2: /RJ45/SchieberegisterInput3/D5 -> /RJ45/SchieberegisterInput1/D4
- R45 pad 2: /RJ45/SchieberegisterInput3/D4 -> /RJ45/SchieberegisterInput1/D3
- R46 pad 2: /RJ45/SchieberegisterInput3/D3 -> /RJ45/SchieberegisterInput1/D2
- R47 pad 2: /RJ45/SchieberegisterInput3/D2 -> /RJ45/SchieberegisterInput1/D1
- R48 pad 2: /RJ45/SchieberegisterInput3/D1 -> /RJ45/SchieberegisterInput1/D0
- R49 pad 2: /RJ45/SchieberegisterInput3/D0 -> /RJ45/SchieberegisterInput3/D7
- R5 pad 1: Net-(U3-QB) -> Net-(U1-QE)
- R5 pad 2: /OutputShift/Out1 -> /OutputShift1/Out4
- R50 pad 2: /RJ45/SchieberegisterInput4/D7 -> /RJ45/SchieberegisterInput3/D6
- R51 pad 2: /RJ45/SchieberegisterInput4/D6 -> /RJ45/SchieberegisterInput3/D5
- R52 pad 2: /RJ45/SchieberegisterInput4/D5 -> /RJ45/SchieberegisterInput3/D4
- R53 pad 2: /RJ45/SchieberegisterInput4/D4 -> /RJ45/SchieberegisterInput3/D3
- R54 pad 2: /RJ45/SchieberegisterInput4/D3 -> /RJ45/SchieberegisterInput3/D2
- R55 pad 2: /RJ45/SchieberegisterInput4/D2 -> /RJ45/SchieberegisterInput3/D1
- R56 pad 2: /RJ45/SchieberegisterInput4/D1 -> /RJ45/SchieberegisterInput3/D0
- R57 pad 2: /RJ45/SchieberegisterInput4/D0 -> /RJ45/SchieberegisterInput4/D7
- R58 pad 2: /RJ45/SchieberegisterInput6/D7 -> /RJ45/SchieberegisterInput4/D6
- R59 pad 2: /RJ45/SchieberegisterInput6/D6 -> /RJ45/SchieberegisterInput4/D5
- R6 pad 1: Net-(U2-QB) -> Net-(U1-QF)
- R6 pad 2: /OutputShift2/Out1 -> /OutputShift1/Out5
- R60 pad 2: /RJ45/SchieberegisterInput6/D5 -> /RJ45/SchieberegisterInput4/D4
- R61 pad 2: /RJ45/SchieberegisterInput6/D4 -> /RJ45/SchieberegisterInput4/D3
- R62 pad 2: /RJ45/SchieberegisterInput6/D3 -> /RJ45/SchieberegisterInput4/D2
- R63 pad 2: /RJ45/SchieberegisterInput6/D2 -> /RJ45/SchieberegisterInput4/D1
- R64 pad 2: /RJ45/SchieberegisterInput6/D1 -> /RJ45/SchieberegisterInput4/D0
- R65 pad 2: /RJ45/SchieberegisterInput6/D0 -> /RJ45/SchieberegisterInput5/D7
- R66 pad 2: /RJ45/SchieberegisterInput5/D7 -> /RJ45/SchieberegisterInput5/D6
- R67 pad 2: /RJ45/SchieberegisterInput5/D6 -> /RJ45/SchieberegisterInput5/D5
- R68 pad 2: /RJ45/SchieberegisterInput5/D5 -> /RJ45/SchieberegisterInput5/D4
- R69 pad 2: /RJ45/SchieberegisterInput5/D4 -> /RJ45/SchieberegisterInput5/D3
- R7 pad 1: Net-(U1-QC) -> Net-(U1-QG)
- R7 pad 2: /OutputShift1/Out2 -> /OutputShift1/Out6
- R70 pad 2: /RJ45/SchieberegisterInput5/D3 -> /RJ45/SchieberegisterInput5/D2
- R71 pad 2: /RJ45/SchieberegisterInput5/D2 -> /RJ45/SchieberegisterInput5/D1
- R72 pad 2: /RJ45/SchieberegisterInput5/D1 -> /RJ45/SchieberegisterInput5/D0
- R73 pad 2: /RJ45/SchieberegisterInput5/D0 -> /RJ45/SchieberegisterInput6/D7
- R74 pad 2: /RJ45/SchieberegisterInput7/D7 -> /RJ45/SchieberegisterInput6/D6
- R75 pad 2: /RJ45/SchieberegisterInput7/D6 -> /RJ45/SchieberegisterInput6/D5
- R76 pad 2: /RJ45/SchieberegisterInput7/D5 -> /RJ45/SchieberegisterInput6/D4
- R77 pad 2: /RJ45/SchieberegisterInput7/D4 -> /RJ45/SchieberegisterInput6/D3
- R78 pad 2: /RJ45/SchieberegisterInput7/D3 -> /RJ45/SchieberegisterInput6/D2
- R79 pad 2: /RJ45/SchieberegisterInput7/D2 -> /RJ45/SchieberegisterInput6/D1
- R8 pad 1: Net-(U3-QC) -> Net-(U1-QH)
- R8 pad 2: /OutputShift/Out2 -> /OutputShift1/Out7
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Routing:
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- added copper zone on In2.Cu, net +5V
- added copper zone on In1.Cu, net GND

Commit message: set Komponents SensorBoard
Parts:
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Connections:
- C10 pad 1: /RJ45/SchieberegisterInput/D2 -> /RJ45/SchieberegisterInput/D1
- C100 pad 1: /RJ45/SchieberegisterInput10/D2 -> /RJ45/SchieberegisterInput10/D1
- C101 pad 1: /RJ45/SchieberegisterInput10/D1 -> /RJ45/SchieberegisterInput10/D2
- C102 pad 1: /RJ45/SchieberegisterInput10/D0 -> /RJ45/SchieberegisterInput10/D3
- C104 pad 1: /RJ45/SchieberegisterInput11/D7 -> /RJ45/SchieberegisterInput11/D4
- C105 pad 1: /RJ45/SchieberegisterInput11/D6 -> /RJ45/SchieberegisterInput11/D5
- C106 pad 1: /RJ45/SchieberegisterInput11/D5 -> /RJ45/SchieberegisterInput11/D6
- C107 pad 1: /RJ45/SchieberegisterInput11/D4 -> /RJ45/SchieberegisterInput11/D7
- C108 pad 1: /RJ45/SchieberegisterInput11/D3 -> /RJ45/SchieberegisterInput11/D0
- C109 pad 1: /RJ45/SchieberegisterInput11/D2 -> /RJ45/SchieberegisterInput11/D1
- C11 pad 1: /RJ45/SchieberegisterInput/D1 -> /RJ45/SchieberegisterInput/D2
- C110 pad 1: /RJ45/SchieberegisterInput11/D1 -> /RJ45/SchieberegisterInput11/D2
- C111 pad 1: /RJ45/SchieberegisterInput11/D0 -> /RJ45/SchieberegisterInput11/D3
- C12 pad 1: /RJ45/SchieberegisterInput/D0 -> /RJ45/SchieberegisterInput/D3
- C14 pad 1: /RJ45/SchieberegisterInput2/D7 -> /RJ45/SchieberegisterInput2/D4
- C15 pad 1: /RJ45/SchieberegisterInput2/D6 -> /RJ45/SchieberegisterInput2/D5
- C16 pad 1: /RJ45/SchieberegisterInput2/D5 -> /RJ45/SchieberegisterInput2/D6
- C17 pad 1: /RJ45/SchieberegisterInput2/D4 -> /RJ45/SchieberegisterInput2/D7
- C18 pad 1: /RJ45/SchieberegisterInput2/D3 -> /RJ45/SchieberegisterInput2/D0
- C19 pad 1: /RJ45/SchieberegisterInput2/D2 -> /RJ45/SchieberegisterInput2/D1
- C20 pad 1: /RJ45/SchieberegisterInput2/D1 -> /RJ45/SchieberegisterInput2/D2
- C21 pad 1: /RJ45/SchieberegisterInput2/D0 -> /RJ45/SchieberegisterInput2/D3
- C23 pad 1: /RJ45/SchieberegisterInput1/D7 -> /RJ45/SchieberegisterInput1/D4
- C24 pad 1: /RJ45/SchieberegisterInput1/D6 -> /RJ45/SchieberegisterInput1/D5
- C25 pad 1: /RJ45/SchieberegisterInput1/D5 -> /RJ45/SchieberegisterInput1/D6
- C26 pad 1: /RJ45/SchieberegisterInput1/D4 -> /RJ45/SchieberegisterInput1/D7
- C27 pad 1: /RJ45/SchieberegisterInput1/D3 -> /RJ45/SchieberegisterInput1/D0
- C28 pad 1: /RJ45/SchieberegisterInput1/D2 -> /RJ45/SchieberegisterInput1/D1
- C29 pad 1: /RJ45/SchieberegisterInput1/D1 -> /RJ45/SchieberegisterInput1/D2
- C30 pad 1: /RJ45/SchieberegisterInput1/D0 -> /RJ45/SchieberegisterInput1/D3
- C32 pad 1: /RJ45/SchieberegisterInput3/D7 -> /RJ45/SchieberegisterInput3/D4
- C33 pad 1: /RJ45/SchieberegisterInput3/D6 -> /RJ45/SchieberegisterInput3/D5
- C34 pad 1: /RJ45/SchieberegisterInput3/D5 -> /RJ45/SchieberegisterInput3/D6
- C35 pad 1: /RJ45/SchieberegisterInput3/D4 -> /RJ45/SchieberegisterInput3/D7
- C36 pad 1: /RJ45/SchieberegisterInput3/D3 -> /RJ45/SchieberegisterInput3/D0
- C37 pad 1: /RJ45/SchieberegisterInput3/D2 -> /RJ45/SchieberegisterInput3/D1
- C38 pad 1: /RJ45/SchieberegisterInput3/D1 -> /RJ45/SchieberegisterInput3/D2
- C39 pad 1: /RJ45/SchieberegisterInput3/D0 -> /RJ45/SchieberegisterInput3/D3
- C41 pad 1: /RJ45/SchieberegisterInput4/D7 -> /RJ45/SchieberegisterInput4/D4
- C42 pad 1: /RJ45/SchieberegisterInput4/D6 -> /RJ45/SchieberegisterInput4/D5
- C43 pad 1: /RJ45/SchieberegisterInput4/D5 -> /RJ45/SchieberegisterInput4/D6
- C44 pad 1: /RJ45/SchieberegisterInput4/D4 -> /RJ45/SchieberegisterInput4/D7
- C45 pad 1: /RJ45/SchieberegisterInput4/D3 -> /RJ45/SchieberegisterInput4/D0
- C46 pad 1: /RJ45/SchieberegisterInput4/D2 -> /RJ45/SchieberegisterInput4/D1
- C47 pad 1: /RJ45/SchieberegisterInput4/D1 -> /RJ45/SchieberegisterInput4/D2
- C48 pad 1: /RJ45/SchieberegisterInput4/D0 -> /RJ45/SchieberegisterInput4/D3
- C5 pad 1: /RJ45/SchieberegisterInput/D7 -> /RJ45/SchieberegisterInput/D4
- C50 pad 1: /RJ45/SchieberegisterInput5/D7 -> /RJ45/SchieberegisterInput5/D4
- C51 pad 1: /RJ45/SchieberegisterInput5/D6 -> /RJ45/SchieberegisterInput5/D5
- C52 pad 1: /RJ45/SchieberegisterInput5/D5 -> /RJ45/SchieberegisterInput5/D6
- C53 pad 1: /RJ45/SchieberegisterInput5/D4 -> /RJ45/SchieberegisterInput5/D7
- C54 pad 1: /RJ45/SchieberegisterInput5/D3 -> /RJ45/SchieberegisterInput5/D0
- C55 pad 1: /RJ45/SchieberegisterInput5/D2 -> /RJ45/SchieberegisterInput5/D1
- C56 pad 1: /RJ45/SchieberegisterInput5/D1 -> /RJ45/SchieberegisterInput5/D2
- C57 pad 1: /RJ45/SchieberegisterInput5/D0 -> /RJ45/SchieberegisterInput5/D3
- C59 pad 1: /RJ45/SchieberegisterInput6/D7 -> /RJ45/SchieberegisterInput6/D4
- C6 pad 1: /RJ45/SchieberegisterInput/D6 -> /RJ45/SchieberegisterInput/D5
- C60 pad 1: /RJ45/SchieberegisterInput6/D6 -> /RJ45/SchieberegisterInput6/D5
- C61 pad 1: /RJ45/SchieberegisterInput6/D5 -> /RJ45/SchieberegisterInput6/D6
- C62 pad 1: /RJ45/SchieberegisterInput6/D4 -> /RJ45/SchieberegisterInput6/D7
- C63 pad 1: /RJ45/SchieberegisterInput6/D3 -> /RJ45/SchieberegisterInput6/D0
- C64 pad 1: /RJ45/SchieberegisterInput6/D2 -> /RJ45/SchieberegisterInput6/D1
- C65 pad 1: /RJ45/SchieberegisterInput6/D1 -> /RJ45/SchieberegisterInput6/D2
- C66 pad 1: /RJ45/SchieberegisterInput6/D0 -> /RJ45/SchieberegisterInput6/D3
- C68 pad 1: /RJ45/SchieberegisterInput7/D7 -> /RJ45/SchieberegisterInput7/D4
- C69 pad 1: /RJ45/SchieberegisterInput7/D6 -> /RJ45/SchieberegisterInput7/D5
- C7 pad 1: /RJ45/SchieberegisterInput/D5 -> /RJ45/SchieberegisterInput/D6
- C70 pad 1: /RJ45/SchieberegisterInput7/D5 -> /RJ45/SchieberegisterInput7/D6
- C71 pad 1: /RJ45/SchieberegisterInput7/D4 -> /RJ45/SchieberegisterInput7/D7
- C72 pad 1: /RJ45/SchieberegisterInput7/D3 -> /RJ45/SchieberegisterInput7/D0
- C73 pad 1: /RJ45/SchieberegisterInput7/D2 -> /RJ45/SchieberegisterInput7/D1
- C74 pad 1: /RJ45/SchieberegisterInput7/D1 -> /RJ45/SchieberegisterInput7/D2
- C75 pad 1: /RJ45/SchieberegisterInput7/D0 -> /RJ45/SchieberegisterInput7/D3
- C77 pad 1: /RJ45/SchieberegisterInput8/D7 -> /RJ45/SchieberegisterInput8/D4
- C78 pad 1: /RJ45/SchieberegisterInput8/D6 -> /RJ45/SchieberegisterInput8/D5
- C79 pad 1: /RJ45/SchieberegisterInput8/D5 -> /RJ45/SchieberegisterInput8/D6
- C8 pad 1: /RJ45/SchieberegisterInput/D4 -> /RJ45/SchieberegisterInput/D7
- C80 pad 1: /RJ45/SchieberegisterInput8/D4 -> /RJ45/SchieberegisterInput8/D7
- C81 pad 1: /RJ45/SchieberegisterInput8/D3 -> /RJ45/SchieberegisterInput8/D0
- C82 pad 1: /RJ45/SchieberegisterInput8/D2 -> /RJ45/SchieberegisterInput8/D1
- C83 pad 1: /RJ45/SchieberegisterInput8/D1 -> /RJ45/SchieberegisterInput8/D2
- C84 pad 1: /RJ45/SchieberegisterInput8/D0 -> /RJ45/SchieberegisterInput8/D3
- C86 pad 1: /RJ45/SchieberegisterInput9/D7 -> /RJ45/SchieberegisterInput9/D4
- C87 pad 1: /RJ45/SchieberegisterInput9/D6 -> /RJ45/SchieberegisterInput9/D5
- C88 pad 1: /RJ45/SchieberegisterInput9/D5 -> /RJ45/SchieberegisterInput9/D6
- C89 pad 1: /RJ45/SchieberegisterInput9/D4 -> /RJ45/SchieberegisterInput9/D7
- C9 pad 1: /RJ45/SchieberegisterInput/D3 -> /RJ45/SchieberegisterInput/D0
- C90 pad 1: /RJ45/SchieberegisterInput9/D3 -> /RJ45/SchieberegisterInput9/D0
- C91 pad 1: /RJ45/SchieberegisterInput9/D2 -> /RJ45/SchieberegisterInput9/D1
- C92 pad 1: /RJ45/SchieberegisterInput9/D1 -> /RJ45/SchieberegisterInput9/D2
- C93 pad 1: /RJ45/SchieberegisterInput9/D0 -> /RJ45/SchieberegisterInput9/D3
- C95 pad 1: /RJ45/SchieberegisterInput10/D7 -> /RJ45/SchieberegisterInput10/D4
- C96 pad 1: /RJ45/SchieberegisterInput10/D6 -> /RJ45/SchieberegisterInput10/D5
- C97 pad 1: /RJ45/SchieberegisterInput10/D5 -> /RJ45/SchieberegisterInput10/D6
- C98 pad 1: /RJ45/SchieberegisterInput10/D4 -> /RJ45/SchieberegisterInput10/D7
- C99 pad 1: /RJ45/SchieberegisterInput10/D3 -> /RJ45/SchieberegisterInput10/D0
- R100 pad 2: /RJ45/SchieberegisterInput9/D4 -> /RJ45/SchieberegisterInput9/D7
- R101 pad 2: /RJ45/SchieberegisterInput9/D3 -> /RJ45/SchieberegisterInput9/D0
- R102 pad 2: /RJ45/SchieberegisterInput9/D2 -> /RJ45/SchieberegisterInput9/D1
- R103 pad 2: /RJ45/SchieberegisterInput9/D1 -> /RJ45/SchieberegisterInput9/D2
- R104 pad 2: /RJ45/SchieberegisterInput9/D0 -> /RJ45/SchieberegisterInput9/D3
- R105 pad 2: /RJ45/SchieberegisterInput10/D7 -> /RJ45/SchieberegisterInput10/D4
- R106 pad 2: /RJ45/SchieberegisterInput10/D6 -> /RJ45/SchieberegisterInput10/D5
- R107 pad 2: /RJ45/SchieberegisterInput10/D5 -> /RJ45/SchieberegisterInput10/D6
- R108 pad 2: /RJ45/SchieberegisterInput10/D4 -> /RJ45/SchieberegisterInput10/D7
- R109 pad 2: /RJ45/SchieberegisterInput10/D3 -> /RJ45/SchieberegisterInput10/D0
- R110 pad 2: /RJ45/SchieberegisterInput10/D2 -> /RJ45/SchieberegisterInput10/D1
- R111 pad 2: /RJ45/SchieberegisterInput10/D1 -> /RJ45/SchieberegisterInput10/D2
- R112 pad 2: /RJ45/SchieberegisterInput10/D0 -> /RJ45/SchieberegisterInput10/D3
- R113 pad 2: /RJ45/SchieberegisterInput11/D7 -> /RJ45/SchieberegisterInput11/D4
- R114 pad 2: /RJ45/SchieberegisterInput11/D6 -> /RJ45/SchieberegisterInput11/D5
- R115 pad 2: /RJ45/SchieberegisterInput11/D5 -> /RJ45/SchieberegisterInput11/D6
- R116 pad 2: /RJ45/SchieberegisterInput11/D4 -> /RJ45/SchieberegisterInput11/D7
- R117 pad 2: /RJ45/SchieberegisterInput11/D3 -> /RJ45/SchieberegisterInput11/D0
- R118 pad 2: /RJ45/SchieberegisterInput11/D2 -> /RJ45/SchieberegisterInput11/D1
- R119 pad 2: /RJ45/SchieberegisterInput11/D1 -> /RJ45/SchieberegisterInput11/D2
- R120 pad 2: /RJ45/SchieberegisterInput11/D0 -> /RJ45/SchieberegisterInput11/D3
- R25 pad 2: /RJ45/SchieberegisterInput/D7 -> /RJ45/SchieberegisterInput/D4
- R26 pad 2: /RJ45/SchieberegisterInput/D6 -> /RJ45/SchieberegisterInput/D5
- R27 pad 2: /RJ45/SchieberegisterInput/D5 -> /RJ45/SchieberegisterInput/D6
- R28 pad 2: /RJ45/SchieberegisterInput/D4 -> /RJ45/SchieberegisterInput/D7
- R29 pad 2: /RJ45/SchieberegisterInput/D3 -> /RJ45/SchieberegisterInput/D0
- R30 pad 2: /RJ45/SchieberegisterInput/D2 -> /RJ45/SchieberegisterInput/D1
- R31 pad 2: /RJ45/SchieberegisterInput/D1 -> /RJ45/SchieberegisterInput/D2
- R32 pad 2: /RJ45/SchieberegisterInput/D0 -> /RJ45/SchieberegisterInput/D3
- R33 pad 2: /RJ45/SchieberegisterInput2/D7 -> /RJ45/SchieberegisterInput2/D4
- R34 pad 2: /RJ45/SchieberegisterInput2/D6 -> /RJ45/SchieberegisterInput2/D5
- R35 pad 2: /RJ45/SchieberegisterInput2/D5 -> /RJ45/SchieberegisterInput2/D6
- R36 pad 2: /RJ45/SchieberegisterInput2/D4 -> /RJ45/SchieberegisterInput2/D7
- R37 pad 2: /RJ45/SchieberegisterInput2/D3 -> /RJ45/SchieberegisterInput2/D0
- R38 pad 2: /RJ45/SchieberegisterInput2/D2 -> /RJ45/SchieberegisterInput2/D1
- R39 pad 2: /RJ45/SchieberegisterInput2/D1 -> /RJ45/SchieberegisterInput2/D2
- R40 pad 2: /RJ45/SchieberegisterInput2/D0 -> /RJ45/SchieberegisterInput2/D3
- R41 pad 2: /RJ45/SchieberegisterInput1/D7 -> /RJ45/SchieberegisterInput1/D4
- R42 pad 2: /RJ45/SchieberegisterInput1/D6 -> /RJ45/SchieberegisterInput1/D5
- R43 pad 2: /RJ45/SchieberegisterInput1/D5 -> /RJ45/SchieberegisterInput1/D6
- R44 pad 2: /RJ45/SchieberegisterInput1/D4 -> /RJ45/SchieberegisterInput1/D7
- R45 pad 2: /RJ45/SchieberegisterInput1/D3 -> /RJ45/SchieberegisterInput1/D0
- R46 pad 2: /RJ45/SchieberegisterInput1/D2 -> /RJ45/SchieberegisterInput1/D1
- R47 pad 2: /RJ45/SchieberegisterInput1/D1 -> /RJ45/SchieberegisterInput1/D2
- R48 pad 2: /RJ45/SchieberegisterInput1/D0 -> /RJ45/SchieberegisterInput1/D3
- R49 pad 2: /RJ45/SchieberegisterInput3/D7 -> /RJ45/SchieberegisterInput3/D4
- R50 pad 2: /RJ45/SchieberegisterInput3/D6 -> /RJ45/SchieberegisterInput3/D5
- R51 pad 2: /RJ45/SchieberegisterInput3/D5 -> /RJ45/SchieberegisterInput3/D6
- R52 pad 2: /RJ45/SchieberegisterInput3/D4 -> /RJ45/SchieberegisterInput3/D7
- R53 pad 2: /RJ45/SchieberegisterInput3/D3 -> /RJ45/SchieberegisterInput3/D0
- R54 pad 2: /RJ45/SchieberegisterInput3/D2 -> /RJ45/SchieberegisterInput3/D1
- R55 pad 2: /RJ45/SchieberegisterInput3/D1 -> /RJ45/SchieberegisterInput3/D2
- R56 pad 2: /RJ45/SchieberegisterInput3/D0 -> /RJ45/SchieberegisterInput3/D3
- R57 pad 2: /RJ45/SchieberegisterInput4/D7 -> /RJ45/SchieberegisterInput4/D4
- R58 pad 2: /RJ45/SchieberegisterInput4/D6 -> /RJ45/SchieberegisterInput4/D5
- R59 pad 2: /RJ45/SchieberegisterInput4/D5 -> /RJ45/SchieberegisterInput4/D6
- R60 pad 2: /RJ45/SchieberegisterInput4/D4 -> /RJ45/SchieberegisterInput4/D7
- R61 pad 2: /RJ45/SchieberegisterInput4/D3 -> /RJ45/SchieberegisterInput4/D0
- R62 pad 2: /RJ45/SchieberegisterInput4/D2 -> /RJ45/SchieberegisterInput4/D1
- R63 pad 2: /RJ45/SchieberegisterInput4/D1 -> /RJ45/SchieberegisterInput4/D2
- R64 pad 2: /RJ45/SchieberegisterInput4/D0 -> /RJ45/SchieberegisterInput4/D3
- R65 pad 2: /RJ45/SchieberegisterInput5/D7 -> /RJ45/SchieberegisterInput5/D4
- R66 pad 2: /RJ45/SchieberegisterInput5/D6 -> /RJ45/SchieberegisterInput5/D5
- R67 pad 2: /RJ45/SchieberegisterInput5/D5 -> /RJ45/SchieberegisterInput5/D6
- R68 pad 2: /RJ45/SchieberegisterInput5/D4 -> /RJ45/SchieberegisterInput5/D7
- R69 pad 2: /RJ45/SchieberegisterInput5/D3 -> /RJ45/SchieberegisterInput5/D0
- R70 pad 2: /RJ45/SchieberegisterInput5/D2 -> /RJ45/SchieberegisterInput5/D1
- R71 pad 2: /RJ45/SchieberegisterInput5/D1 -> /RJ45/SchieberegisterInput5/D2
- R72 pad 2: /RJ45/SchieberegisterInput5/D0 -> /RJ45/SchieberegisterInput5/D3
- R73 pad 2: /RJ45/SchieberegisterInput6/D7 -> /RJ45/SchieberegisterInput6/D4
- R74 pad 2: /RJ45/SchieberegisterInput6/D6 -> /RJ45/SchieberegisterInput6/D5
- R75 pad 2: /RJ45/SchieberegisterInput6/D5 -> /RJ45/SchieberegisterInput6/D6
- R76 pad 2: /RJ45/SchieberegisterInput6/D4 -> /RJ45/SchieberegisterInput6/D7
- R77 pad 2: /RJ45/SchieberegisterInput6/D3 -> /RJ45/SchieberegisterInput6/D0
- R78 pad 2: /RJ45/SchieberegisterInput6/D2 -> /RJ45/SchieberegisterInput6/D1
- R79 pad 2: /RJ45/SchieberegisterInput6/D1 -> /RJ45/SchieberegisterInput6/D2
- R80 pad 2: /RJ45/SchieberegisterInput6/D0 -> /RJ45/SchieberegisterInput6/D3
- R81 pad 2: /RJ45/SchieberegisterInput7/D7 -> /RJ45/SchieberegisterInput7/D4
- R82 pad 2: /RJ45/SchieberegisterInput7/D6 -> /RJ45/SchieberegisterInput7/D5
- R83 pad 2: /RJ45/SchieberegisterInput7/D5 -> /RJ45/SchieberegisterInput7/D6
- R84 pad 2: /RJ45/SchieberegisterInput7/D4 -> /RJ45/SchieberegisterInput7/D7
- R85 pad 2: /RJ45/SchieberegisterInput7/D3 -> /RJ45/SchieberegisterInput7/D0
- R86 pad 2: /RJ45/SchieberegisterInput7/D2 -> /RJ45/SchieberegisterInput7/D1
- R87 pad 2: /RJ45/SchieberegisterInput7/D1 -> /RJ45/SchieberegisterInput7/D2
- R88 pad 2: /RJ45/SchieberegisterInput7/D0 -> /RJ45/SchieberegisterInput7/D3
- R89 pad 2: /RJ45/SchieberegisterInput8/D7 -> /RJ45/SchieberegisterInput8/D4
- R90 pad 2: /RJ45/SchieberegisterInput8/D6 -> /RJ45/SchieberegisterInput8/D5
- R91 pad 2: /RJ45/SchieberegisterInput8/D5 -> /RJ45/SchieberegisterInput8/D6
- R92 pad 2: /RJ45/SchieberegisterInput8/D4 -> /RJ45/SchieberegisterInput8/D7
- R93 pad 2: /RJ45/SchieberegisterInput8/D3 -> /RJ45/SchieberegisterInput8/D0
- R94 pad 2: /RJ45/SchieberegisterInput8/D2 -> /RJ45/SchieberegisterInput8/D1
- R95 pad 2: /RJ45/SchieberegisterInput8/D1 -> /RJ45/SchieberegisterInput8/D2
- R96 pad 2: /RJ45/SchieberegisterInput8/D0 -> /RJ45/SchieberegisterInput8/D3
- R97 pad 2: /RJ45/SchieberegisterInput9/D7 -> /RJ45/SchieberegisterInput9/D4
- R98 pad 2: /RJ45/SchieberegisterInput9/D6 -> /RJ45/SchieberegisterInput9/D5
- R99 pad 2: /RJ45/SchieberegisterInput9/D5 -> /RJ45/SchieberegisterInput9/D6
- U10 pad 11: /RJ45/SchieberegisterInput6/D0 -> /RJ45/SchieberegisterInput6/D3
- U10 pad 12: /RJ45/SchieberegisterInput6/D1 -> /RJ45/SchieberegisterInput6/D2
- U10 pad 13: /RJ45/SchieberegisterInput6/D2 -> /RJ45/SchieberegisterInput6/D1
- U10 pad 14: /RJ45/SchieberegisterInput6/D3 -> /RJ45/SchieberegisterInput6/D0
- U10 pad 3: /RJ45/SchieberegisterInput6/D4 -> /RJ45/SchieberegisterInput6/D7
- U10 pad 4: /RJ45/SchieberegisterInput6/D5 -> /RJ45/SchieberegisterInput6/D6
- U10 pad 5: /RJ45/SchieberegisterInput6/D6 -> /RJ45/SchieberegisterInput6/D5
- U10 pad 6: /RJ45/SchieberegisterInput6/D7 -> /RJ45/SchieberegisterInput6/D4
- U11 pad 11: /RJ45/SchieberegisterInput7/D0 -> /RJ45/SchieberegisterInput7/D3
- U11 pad 12: /RJ45/SchieberegisterInput7/D1 -> /RJ45/SchieberegisterInput7/D2
- U11 pad 13: /RJ45/SchieberegisterInput7/D2 -> /RJ45/SchieberegisterInput7/D1
- U11 pad 14: /RJ45/SchieberegisterInput7/D3 -> /RJ45/SchieberegisterInput7/D0
- U11 pad 3: /RJ45/SchieberegisterInput7/D4 -> /RJ45/SchieberegisterInput7/D7
- U11 pad 4: /RJ45/SchieberegisterInput7/D5 -> /RJ45/SchieberegisterInput7/D6
- U11 pad 5: /RJ45/SchieberegisterInput7/D6 -> /RJ45/SchieberegisterInput7/D5
- U11 pad 6: /RJ45/SchieberegisterInput7/D7 -> /RJ45/SchieberegisterInput7/D4
- U12 pad 11: /RJ45/SchieberegisterInput8/D0 -> /RJ45/SchieberegisterInput8/D3
- U12 pad 12: /RJ45/SchieberegisterInput8/D1 -> /RJ45/SchieberegisterInput8/D2
- U12 pad 13: /RJ45/SchieberegisterInput8/D2 -> /RJ45/SchieberegisterInput8/D1
- U12 pad 14: /RJ45/SchieberegisterInput8/D3 -> /RJ45/SchieberegisterInput8/D0
- U12 pad 3: /RJ45/SchieberegisterInput8/D4 -> /RJ45/SchieberegisterInput8/D7
- U12 pad 4: /RJ45/SchieberegisterInput8/D5 -> /RJ45/SchieberegisterInput8/D6
- U12 pad 5: /RJ45/SchieberegisterInput8/D6 -> /RJ45/SchieberegisterInput8/D5
- U12 pad 6: /RJ45/SchieberegisterInput8/D7 -> /RJ45/SchieberegisterInput8/D4
- U13 pad 11: /RJ45/SchieberegisterInput9/D0 -> /RJ45/SchieberegisterInput9/D3
- U13 pad 12: /RJ45/SchieberegisterInput9/D1 -> /RJ45/SchieberegisterInput9/D2
- U13 pad 13: /RJ45/SchieberegisterInput9/D2 -> /RJ45/SchieberegisterInput9/D1
- U13 pad 14: /RJ45/SchieberegisterInput9/D3 -> /RJ45/SchieberegisterInput9/D0
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Routing:
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
Commit message: finish SensBoard
Parts:
- removed C10, C100, C101, C102, C104, C105, C106, C107, C108, C109, C11, C110, C111, C12, C14, C15, C16, C17, C18, C19, C20, C21, C23, C24, C25, C26, C27, C28, C29, C30, C32, C33, C34, C35, C36, C37, C38, C39, C41, C42, C43, C44, C45, C46, C47, C48, C5, C50, C51, C52, C53, C54, C55, C56, C57, C59, C6, C60, C61, C62, C63, C64, C65, C66, C68, C69, C7, C70, C71, C72, C73, C74, C75, C77, C78, C79, C8, C80, C81, C82, C83, C84, C86, C87, C88, C89, C9, C90, C91, C92, C93, C95, C96, C97, C98, C99: 100n, Capacitor_SMD:C_0402_1005Metric
- added H1: MountingHole, MountingHole:MountingHole_3.2mm_M3, F.Cu at (65.6, 114.3)
- added H2: MountingHole, MountingHole:MountingHole_3.2mm_M3, F.Cu at (84.6, 114.3)
- added H3: MountingHole, MountingHole:MountingHole_3.2mm_M3, F.Cu at (127.1, 77.2)
- added H4: MountingHole, MountingHole:MountingHole_3.2mm_M3, F.Cu at (127.1, 85.1)
- J1, J2: footprint Connector_JST:JST_PH_B8B-PH-SM4-TB_1x08-1MP_P2.00mm_Vertical -> Connector_JST:JST_PH_B9B-PH-SM4-TB_1x09-1MP_P2.00mm_Vertical
- moved R108 164.3 mm to (35.0, 74.8), turned to -90 degrees
- moved R107 162.7 mm to (35.0, 77.1), turned to -90 degrees
- moved R106 160.8 mm to (35.0, 79.4), turned to 90 degrees
- moved R105 158.8 mm to (35.0, 81.7), turned to 90 degrees
- moved C94 156.8 mm to (43.8, 72.4), turned to 0 degrees
- moved U14 155.7 mm to (40.1, 78.3), turned to 0 degrees
- moved R120 154.1 mm to (35.0, 88.7), turned to -90 degrees
- moved R109 153.0 mm to (45.1, 74.8), turned to -90 degrees
- moved R119 152.2 mm to (35.0, 91.0), turned to -90 degrees
- moved R110 151.0 mm to (45.1, 77.1), turned to -90 degrees
- moved R118 150.8 mm to (35.0, 93.2), turned to 90 degrees
- moved R117 149.1 mm to (35.0, 95.5), turned to 90 degrees
- moved R111 148.8 mm to (45.1, 79.4), turned to 90 degrees
- moved R92 148.2 mm to (49.3, 74.8), turned to -90 degrees
- moved R112 146.9 mm to (45.1, 81.7), turned to 90 degrees
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Connections:
- J2 pad 1: +5V -> GND
- J2 pad 2: Data_Output -> Led_Clk
- J2 pad 3: Data_Latch -> Led_Latch
- J2 pad 4: Data_Clk -> Led_OE
- J2 pad 6: Led_OE -> Data_Clk
- J2 pad 7: Led_Latch -> Data_Latch
- J2 pad 8: Led_Clk -> Data_Output
Routing:
- net Data_Clk: track 1.10 -> 228.3 mm, vias 1 -> 12
- net Data_Latch: track 1.10 -> 219.7 mm, vias 1 -> 12
- net Led_Clk: track 0.00 -> 163.5 mm
- net Led_OE: track 0.00 -> 88.7 mm, vias 0 -> 5
- net +5V: track 21.0 -> 108.0 mm, vias 20 -> 112
- net Led_Latch: track 0.00 -> 86.5 mm, vias 0 -> 5
- net /OutputShift2/Out3: track 0.00 -> 77.2 mm, vias 0 -> 1
- net /OutputShift/Out6: track 0.00 -> 76.5 mm, vias 0 -> 1
- net /OutputShift2/Out7: track 0.00 -> 75.7 mm, vias 0 -> 1
- net /OutputShift/Out2: track 0.00 -> 70.3 mm, vias 0 -> 1
- net /OutputShift2/Out2: track 0.00 -> 66.5 mm, vias 0 -> 1
- net /OutputShift1/Out7: track 0.00 -> 65.1 mm, vias 0 -> 1
- net /OutputShift1/Out6: track 0.00 -> 64.8 mm, vias 0 -> 1
- net /OutputShift1/Out2: track 0.00 -> 64.7 mm, vias 0 -> 1
- net /OutputShift/Out3: track 0.00 -> 64.0 mm, vias 0 -> 1
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Other:
- board size 200 x 100 mm -> 87 x 84 mm

Commit message: add pull UP/DOWN
Parts:
- removed H3, H4: MountingHole, MountingHole:MountingHole_3.2mm_M3
- added R121: 0, Resistor_SMD:R_0402_1005Metric, F.Cu at (115.6, 74.8)
- added R122: 0, Resistor_SMD:R_0402_1005Metric, F.Cu at (102.3, 74.8)
- added R123: 0, Resistor_SMD:R_0402_1005Metric, F.Cu at (106.9, 100.0)
- added R124: 0, Resistor_SMD:R_0402_1005Metric, F.Cu at (96.0, 98.3)
- added R125: 0, Resistor_SMD:R_0402_1005Metric, F.Cu at (88.1, 74.8)
- added R126: 0, Resistor_SMD:R_0402_1005Metric, F.Cu at (81.7, 98.3)
- added R127: 0, Resistor_SMD:R_0402_1005Metric, F.Cu at (74.4, 74.8)
- added R128: 0, Resistor_SMD:R_0402_1005Metric, F.Cu at (68.0, 98.3)
- added R129: 0, Resistor_SMD:R_0402_1005Metric, F.Cu at (60.4, 74.8)
- added R130: 0, Resistor_SMD:R_0402_1005Metric, F.Cu at (54.0, 98.3)
- added R131: 0, Resistor_SMD:R_0402_1005Metric, F.Cu at (46.2, 74.8)
- added R132: 0, Resistor_SMD:R_0402_1005Metric, F.Cu at (39.8, 98.3)
- added R133: 0, Resistor_SMD:R_0402_1005Metric, F.Cu at (72.0, 118.1)
- added R134: 0, Resistor_SMD:R_0402_1005Metric, F.Cu at (52.4, 117.9)
- added R135: 0, Resistor_SMD:R_0402_1005Metric, F.Cu at (91.9, 118.3)
- R1, R10, R11, R12, R13, R14, R15, R16, R17, R18, R19, R2, R20, R21, R22, R23, R24, R3, R4, R5, R6, R7, R8, R9: value R -> 120
Connections:
- U1 pad 10: unconnected-(U1-~{SRCLR}-Pad10) -> Net-(U1-~{SRCLR})
- U10 pad 15: unconnected-(U10-~{CE}-Pad15) -> Net-(U10-~{CE})
- U11 pad 15: unconnected-(U11-~{CE}-Pad15) -> Net-(U11-~{CE})
- U12 pad 15: unconnected-(U12-~{CE}-Pad15) -> Net-(U12-~{CE})
- U13 pad 15: unconnected-(U13-~{CE}-Pad15) -> Net-(U13-~{CE})
- U14 pad 15: unconnected-(U14-~{CE}-Pad15) -> Net-(U14-~{CE})
- U15 pad 15: unconnected-(U15-~{CE}-Pad15) -> Net-(U15-~{CE})
- U2 pad 10: unconnected-(U2-~{SRCLR}-Pad10) -> Net-(U2-~{SRCLR})
- U3 pad 10: unconnected-(U3-~{SRCLR}-Pad10) -> Net-(U3-~{SRCLR})
- U4 pad 15: unconnected-(U4-~{CE}-Pad15) -> Net-(U4-~{CE})
- U5 pad 15: unconnected-(U5-~{CE}-Pad15) -> Net-(U5-~{CE})
- U6 pad 15: unconnected-(U6-~{CE}-Pad15) -> Net-(U6-~{CE})
- U7 pad 15: unconnected-(U7-~{CE}-Pad15) -> Net-(U7-~{CE})
- U8 pad 15: unconnected-(U8-~{CE}-Pad15) -> Net-(U8-~{CE})
- U9 pad 15: unconnected-(U9-~{CE}-Pad15) -> Net-(U9-~{CE})
Routing:
- net Net-(U5-~{CE}): track 0.00 -> 6.21 mm
- net Net-(U9-~{CE}): track 0.00 -> 5.59 mm
- net Net-(U7-~{CE}): track 0.00 -> 5.37 mm
- net Net-(U15-~{CE}): track 0.00 -> 5.32 mm
- net Net-(U13-~{CE}): track 0.00 -> 5.29 mm
- net Net-(U11-~{CE}): track 0.00 -> 5.22 mm
- net GND: track 32.0 -> 36.2 mm, vias 40 -> 39
- net Net-(U10-~{CE}): track 0.00 -> 3.25 mm
- net Net-(U6-~{CE}): track 0.00 -> 3.24 mm
- net Net-(U8-~{CE}): track 0.00 -> 3.24 mm
- net Net-(U12-~{CE}): track 0.00 -> 3.24 mm
- net Net-(U14-~{CE}): track 0.00 -> 3.20 mm
- net Net-(U4-~{CE}): track 0.00 -> 3.18 mm
- net +5V: track 108.0 -> 110.3 mm, vias 112 -> 115
- net Net-(U3-~{SRCLR}): track 0.00 -> 1.65 mm
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