File: Id_Board/Id_Board.kicad_sch (KiCad schematic)
At the start: 14 parts, among them J1 RJ45, J10 RJ45, J2 Conn_01x02_Pin, J3 Conn_01x02_Pin, J4 RJ45, J5 RJ45, J6 RJ45, J7 RJ45, J8 RJ45, J9 RJ45

Commit message: finished IdBoard
Parts:
- removed J1, J10, J4, J5, J6, J7, J8, J9: RJ45, symbol Connector:RJ45
- added J1: (no value), LCSC:RJ45-TH_HC-WK88-H13-1X8-55QS_1, symbol Techbeard:RJ45-8
- added R1, R10, R11, R12, R13, R14, R15, R16, R17, R18, R19, R2, R20, R21, R22, R23, R24, R3, R4, R5, R6, R7, R8, R9: 0, Resistor_SMD:R_0603_1608Metric, symbol Device:R
- added SW1: SW_DIP_x08, LCSC:SW-SMD_16P-L20.3-W6.0-P2.54-LS9.3-BL, symbol Switch:SW_DIP_x08
- H1, H2, H3, H4: footprint (none) -> MountingHole:MountingHole_3.2mm_M3
- J2, J3: footprint (none) -> Connector_JST:JST_PH_B2B-PH-SM4-TB_1x02-1MP_P2.00mm_Vertical
Connections:
- net GND: now also R1.1, R10.1, R11.1, R12.1, R13.1, R14.1, R15.1, R16.1, R17.1, R18.1, R19.1, R2.1, R20.1, R21.1, R22.1, R23.1, R24.1, R3.1, R4.1, R5.1, R6.1, R7.1, R8.1, R9.1, SW1.1, SW1.2, SW1.3, SW1.4, SW1.5, SW1.6, SW1.7, SW1.8
- new net: J1.D1, R10.2
- new net: J1.A3, R3.2
- new net: J1.H1, R22.2
- new net: J1.E3, R15.2
- new net: J1.B3, R6.2
- new net: J1.D2, R11.2
- new net: J1.C1, R7.2
- new net: J1.C2, R8.2
- new net: J1.D3, R12.2
- new net: J1.A2, R2.2
- new net: J1.G3, R21.2
- new net: J1.E2, R14.2
- new net: J1.G1, R19.2
- new net: J1.G2, R20.2
- new net: J1.E1, R13.2
- new net: J1.F2, R17.2
- new net: J1.B2, R5.2
- new net: J1.A1, R1.2
- new net: J1.C3, R9.2
- new net: J1.F1, R16.2
- new net: J1.H2, R23.2
- new net: J1.H3, R24.2
- new net: J1.B1, R4.2
- new net: J1.F3, R18.2
- new net BoardA: J1.A4, J1.B4, J1.C4, J1.D4, J1.E4, J1.F4, J1.G4, J1.H4, SW1.9
- new net BoardB: J1.A5, J1.B5, J1.C5, J1.D5, J1.E5, J1.F5, J1.G5, J1.H5, SW1.10
- new net BoardC: J1.A6, J1.B6, J1.C6, J1.D6, J1.E6, J1.F6, J1.G6, J1.H6, SW1.11
- new net BoardD: J1.A7, J1.B7, J1.C7, J1.D7, J1.E7, J1.F7, J1.G7, J1.H7, SW1.12
- new net ParityA: J1.A8, J1.C8, J1.E8, J1.G8, SW1.16
- new net ParityB: J1.B8, J1.D8, J1.F8, J1.H8, SW1.15
- no-connect marks 0 -> 2
Other:
- removed sheet Dip
- removed sheet Dip1
- removed sheet Dip2
- removed sheet Dip3
- removed sheet Dip4
- removed sheet Dip5
- removed sheet Dip6
- removed sheet Dip7

Commit message: Production File generate
Parts:
- R1, R12, R13, R14, R17, R19, R2, R3, R5, R6, R7, R9: now left out of the parts list
Changed lines of the file:
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@@
 		(body_style 1)
 		(exclude_from_sim no)
-		(in_bom yes)
+		(in_bom no)
 		(on_board yes)
 		(in_pos_files yes)
@@
 		(body_style 1)
 		(exclude_from_sim no)
-		(in_bom yes)
+		(in_bom no)
 		(on_board yes)
 		(in_pos_files yes)
@@
 		(body_style 1)
 		(exclude_from_sim no)
-		(in_bom yes)
+		(in_bom no)
 		(on_board yes)
 		(in_pos_files yes)
@@
 		(body_style 1)
 		(exclude_from_sim no)
-		(in_bom yes)
+		(in_bom no)
 		(on_board yes)
 		(in_pos_files yes)
@@
 		(body_style 1)
 		(exclude_from_sim no)
-		(in_bom yes)
+		(in_bom no)
 		(on_board yes)
 		(in_pos_files yes)
@@
 		(body_style 1)
 		(exclude_from_sim no)
-		(in_bom yes)
+		(in_bom no)
 		(on_board yes)
 		(in_pos_files yes)
@@
 		(body_style 1)
 		(exclude_from_sim no)
-		(in_bom yes)
+		(in_bom no)
 		(on_board yes)
 		(in_pos_files yes)
@@
 		(body_style 1)
 		(exclude_from_sim no)
-		(in_bom yes)
+		(in_bom no)
 		(on_board yes)
 		(in_pos_files yes)
@@
 		(body_style 1)
 		(exclude_from_sim no)
-		(in_bom yes)
+		(in_bom no)
 		(on_board yes)
 		(in_pos_files yes)
@@
 		(body_style 1)
 		(exclude_from_sim no)
-		(in_bom yes)
+		(in_bom no)
 		(on_board yes)
 		(in_pos_files yes)
@@
 		(body_style 1)
 		(exclude_from_sim no)
-		(in_bom yes)
+		(in_bom no)
 		(on_board yes)
 		(in_pos_files yes)
@@
 		(body_style 1)
 		(exclude_from_sim no)
-		(in_bom yes)
+		(in_bom no)
 		(on_board yes)
 		(in_pos_files yes)
